Commit message: feat(robot_arm_description): 랙피니언 2모터 그리퍼 URDF 이식 및 소비자 설정 갱신
2026_07_16 Fusion360 export의 랙피니언 그리퍼를 현재 Isaac Sim 기반 URDF에
서브트리 단위로 이식하고, 이 이름 체계를 참조하는 설정을 전부 맞췄다.

## URDF (robot_arm_description)

이식 지점은 link_039(5축 모듈 연결부) — 두 export에서 world 포즈 0.000mm,
mesh bbox 오차 0.019mm로 동일 파트임을 확인하고 골랐다. 신규 export는 현재
모델 대비 Rz(180°)+y(-10mm) 좌표계인데, 이 차이는 그래프트 조인트
fixed_joint_036 하나가 전부 흡수하므로 서브트리 내부 origin/axis/limit/
inertial은 원본 export 값 그대로다.

- 옛 평행4절 그리퍼 링크 link_041~057(17개)+조인트 17개 제거
- 신규 링크 link_041~050(10개)+조인트 10개 추가 → 51 link / 50 joint
- 팔 링크(base_link, link_001~040)는 전부 그대로. mesh bbox 0.2mm 이내로
  신규 export에도 동일 파트가 존재함을 확인했다.

그리퍼는 1 DOF다. 서보 2개(id 3,4)를 항상 같은 방향·같은 값으로 돌리므로
gripper_left_pinion_joint 하나만 구동 조인트로 두고 나머지 3개(우 피니언,
좌우 랙)를 전부 여기에 직접 mimic 시켰다(다단 mimic은 KDL이 못 푼다).
mimic multiplier는 export에 없어 직접 산출했다 — 기어 STL 37.91mm/36치 →
모듈 1 → 피치반경 18mm. 맞물림 쌍도 기하로 확정했다(피니언↔랙 각 18.1mm,
교차 조합은 19.6mm).

부호 규약은 실기 기준이다: θ=0이 완전 닫힘, 양수로 갈수록 열림, 상한
1.9444 rad(랙 가동량 35mm). 좌우 조는 항상 대칭으로 움직인다 — 두 랙이
서로 반대 world 축으로 미끄러져서, 조 중심 x=-10.80mm가 전 구간 불변임을
URDF FK로 확인했다.

arm_joint_4 축 이동(world 7.141mm)도 신규 CAD 기준으로 반영했다. 축과 함께
link_038(어댑터)·link_040(XL430_T)만 옮겨가고 나머지는 제자리여야 해서
fixed_joint_025·026·034·arm_joint_5의 local origin을 신규 export의 world
포즈에서 역산해 보정했다.

arm_joint_2·3의 하한은 0으로 되돌렸다(접힘자세 탐색용으로 -10°까지 열어뒀던
미커밋 변경분 원복 — 해당 구간은 자기충돌이 확인된 영역이다).

RViz 설정(rviz/robot_arm.rviz)을 추가하고 display.launch.py가 -d로 넘기게
했다. 저장된 config가 없어 Fixed Frame·RobotModel·Durability를 매번 손으로
잡아야 했다.

## 소비자 설정

- robot_arm.srdf: arm 체인 tip_link link_051 → link_039, gripper 그룹과
  group_state를 새 구동 조인트로, end_effector parent_link도 link_039로.
  disable_collisions의 Adjacent 50쌍은 URDF에서 기계적으로 재생성했고,
  Default는 무효가 된 그리퍼 쌍을 걷어내고 60개 샘플로 재산출해 9쌍을 등록했다.
- joint_limits / initial_positions / ros2_controllers / moveit_controllers /
  ros2_control.xacro: gripper_drive_joint → gripper_left_pinion_joint
- gripper_presets.py: 구동 조인트 교체. 구동 조인트가 prismatic(m)에서
  revolute(rad)로 바뀌었으므로 gripper_open_m/close_m → *_rad 로 개명하고
  값을 URDF 리미트(0 / 1.9444)로 맞췄다. tick 값은 HW-8 단일서보 유산값이라
  미검증 상태로 두고 경고 주석을 달았다.
- moveit_dynamixel_bridge.py: 위 개명 반영, m 도메인 식별자 정리
- arm_fsm_node.py: tip_link 기본값 link_051 → link_039

레거시 dynamixel_position_node.py는 별도 런타임이라 의도적으로 건드리지 않았다.

## 검증

- 가동 조인트 9개 축이 신규 export 대비 위치차 0.00µm / 축차 0.0000°
- 트리 단일 루트, 중복 parent 0, mesh 참조 51/51
- colcon build 6개 패키지 통과
- display.launch.py: 에러 0, /joint_states 9개, /tf_static 41 + /tf 9
- demo.launch.py(mock): 컨트롤러 3개 active, move_group 정상 기동
- 사용자가 RViz에서 전 관절·그리퍼 개폐 육안 확인

home 자세에 link_002/link_026, link_034/link_037 충돌이 남는데 두 쌍 모두
main과 정점거리 0.000mm로 동일한 기존 문제다(SRDF 주석에 기록됨).

Co-Authored-By: Claude Opus 5 <noreply@anthropic.com>

File: ros2_ws/src/robot_arm_description/urdf/robot_arm.urdf (robot description, URDF)
Before this commit: robot robot_arm, 58 links, 57 joints
Links:
- removed link link_051
- removed link link_052
- removed link link_053
- removed link link_054
- removed link link_055
- removed link link_056
- removed link link_057
- link link_041: mass 0.09721724258742875 -> 0.07583994930008672
- link link_042: mass 0.008257662906206078 -> 0.5057750603466008
- link link_043: mass 0.008257662983629954 -> 0.08821021033890362
- link link_044: mass 0.010975108826546717 -> 0.08821021033890375
- link link_045: mass 0.010975108826539954 -> 0.0034506939547765065
- link link_046: mass 0.008257662906252378 -> 0.0034506939547765073
- link link_047: mass 0.008257662983629954 -> 0.009342051864502975
- link link_048: mass 0.015261011971620197 -> 0.009342052845410124
- link link_049: mass 0.07922324071673989 -> 0.14107452059972816
- link link_050: mass 0.015261011971620171 -> 0.14107452059972586
Joints:
- removed joint gripper_drive_joint
- removed joint gripper_left_crank_joint
- removed joint gripper_left_finger_fixed
- removed joint gripper_left_inner_joint
- removed joint gripper_left_lower_jaw_joint
- removed joint gripper_left_upper_jaw_joint
- removed joint gripper_linkage_base_fixed
- removed joint gripper_right_crank_joint
- removed joint gripper_right_finger_fixed
- removed joint gripper_right_inner_joint
- removed joint gripper_right_lower_jaw_joint
- removed joint gripper_right_upper_jaw_joint
- added joint fixed_joint_041: type fixed, parent link_044, child link_046, origin xyz=-0.007999 -0.0039 -0.01175 rpy=0 0 0
- added joint gripper_left_pinion_joint: type revolute, parent link_045, child link_047, origin xyz=0.0 -0.006 0.0 rpy=0 0 0, axis 0.0 -1.0 -0.0, limit lower=0.0 upper=1.9444444444444444 effort=100 velocity=100
- added joint gripper_left_rack_joint: type prismatic, parent link_042, child link_049, origin xyz=-0.098787 -0.259411 0.161136 rpy=0 0 0, axis 1.0 -0.0 -0.0, limit lower=-0.035 upper=0.0 effort=100 velocity=100, mimic joint=gripper_left_pinion_joint multiplier=-0.018 offset=0.0
- added joint gripper_right_pinion_joint: type revolute, parent link_046, child link_048, origin xyz=0.0 -0.004 0.0 rpy=0 0 0, axis -0.0 -1.0 -0.0, limit lower=0.0 upper=1.9444444444444444 effort=100 velocity=100, mimic joint=gripper_left_pinion_joint multiplier=1.0 offset=0.0
- added joint gripper_right_rack_joint: type prismatic, parent link_042, child link_050, origin xyz=-0.109737 -0.047 -0.052497 rpy=0 0 0, axis -1.0 0.0 0.0, limit lower=-0.035 upper=0.0 effort=100 velocity=100, mimic joint=gripper_left_pinion_joint multiplier=-0.018 offset=0.0
- joint arm_joint_4: origin xyz=0.0 0.06337296 0.0 rpy=3.141592653589793 -0.0 3.141592653589793 -> xyz=-0.0045 0.06891702 -0.0001 rpy=3.141592653589793 -0.0 3.141592653589793
- joint arm_joint_5: origin xyz=-0.030999999999999996 0.0007499999999999929 0.003899999999999997 rpy=-1.3358230912699144e-33 -4.09841728479371e-34 0.0 -> xyz=-0.030900000000000004 0.005250000000000009 -0.0016439999999999977 rpy=-1.3358230912699144e-33 -4.09841728479371e-34 0.0
- joint fixed_joint_025: origin xyz=0.0 0.0 0.003999999999999999 rpy=3.141592653589793 -0.0 0.0 -> xyz=-0.004500000000000006 -0.0055439999999999864 0.003900000000000089 rpy=3.141592653589793 -0.0 0.0
- joint fixed_joint_026: origin xyz=0.010500000000000008 0.0 -0.006600000000000002 rpy=0.0 -0.0 0.0 -> xyz=0.006000000000000005 -0.0055439999999999864 -0.006699999999999907 rpy=0.0 -0.0 0.0
- joint fixed_joint_034: origin xyz=-0.004750000000000015 0.095 0.014950000000000001 rpy=-1.5707963267948966 1.5707963267948966 0 -> xyz=-0.0002499999999999845 0.100544 0.015050000000000003 rpy=-1.5707963267948966 1.5707963267948966 0
- joint fixed_joint_036: origin xyz=0.0 0.0 -0.073 rpy=0.0 9.298773838736199e-33 0.0 -> xyz=0.0 0.0 -0.073 rpy=1.5707963267948966 0.0 -3.141592653589793
- joint fixed_joint_037: child link_051 -> link_042; origin xyz=0.0 0.001999999999999993 -0.01 rpy=1.5707963267948966 -1.9721522630525295e-31 1.5707963267948966 -> xyz=0.014 -0.005 0.018 rpy=0 0 0
- joint fixed_joint_038: child link_052 -> link_043; origin xyz=0.0 0.0 0.01 rpy=0.0 -0.0 0.0 -> xyz=-0.002 -0.034 -0.007 rpy=0 0 0; parent link_055 -> link_042
- joint fixed_joint_039: child link_053 -> link_044; origin xyz=0.0 0.0 0.01 rpy=0.0 -0.0 -8.344469655179642e-31 -> xyz=-0.026 -0.034 -0.007 rpy=0 0 0; parent link_056 -> link_042
- joint fixed_joint_040: child link_054 -> link_045; origin xyz=0.0 0.0 0.01 rpy=0.0 -9.860761315262648e-32 -5.551115123125708e-17 -> xyz=0.008001 -0.002 -0.010249 rpy=0 0 0; parent link_057 -> link_043

File: ros2_ws/src/robot_arm_moveit_config/config/robot_arm.ros2_control.xacro (robot description, xacro)
@@ -43,8 +43,8 @@
                 <state_interface name="velocity"/>
             </joint>
-            <joint name="gripper_drive_joint">
+            <joint name="gripper_left_pinion_joint">
                 <command_interface name="position"/>
                 <state_interface name="position">
-                  <param name="initial_value">${initial_positions['gripper_drive_joint']}</param>
+                  <param name="initial_value">${initial_positions['gripper_left_pinion_joint']}</param>
                 </state_interface>
                 <state_interface name="velocity"/>

Commit message: feat(robot_arm_description): 손목 카메라 통합 + 전체 URDF/SRDF 재생성
2026_07_29_랙피니언_URDF_description.zip(base_link~5축 팔~그리퍼~손목카메라 통합
CAD export)로 robot_arm.urdf를 처음부터 다시 생성. 이전 손목 카메라는
camera_tf.launch.py의 홈포즈 고정 static TF placeholder였는데, 이제 URDF
관절 체인(link_036 -> 상단_1/하단_1 브래킷 -> wrist_camera_link)으로 통합돼
팔 자세에 따라 동적으로 TF가 나온다.

- robot_arm.urdf: 전체 52 링크/51 조인트 재생성. arm_joint_1..5 등 시맨틱
  조인트 이름은 유지, 구조 링크는 link_0XX로 재번호. 그리퍼 구동 조인트
  (revolute/mimic, 부호 규약, 리밋)는 2026-07-29 실기 검증값을 자동 생성
  스크립트 위에 수동 패치로 보존.
- robot_arm.srdf: arm 체인 tip_link/end_effector를 link_043(그리퍼 하우징)
  으로 갱신. disable_collisions는 새 URDF에서 Adjacent 51쌍을 기계적으로
  재추출 + /check_state_validity 200샘플 무작위 검증으로 상시-접촉 Default
  쌍 22개(그리퍼 완전닫힘 경계 케이스 2개 포함) 확정.
- arm_fsm_node.py: tip_link 기본값을 SRDF와 동기화(link_039 -> link_043).
- camera_tf.launch.py: 손목 카메라 static TF 발행 제거(URDF가 대체).

MoveIt mock(demo.launch.py)으로 컨트롤러 3개 active + 플래닝 가능 확인.
Adjacent 200샘플 시점에 home/stow(all-zero) 자세 자체에서도 일부 구간
(link_036/038 등, 자세 의존 92%)이 self-collision으로 잡혀 후속 확인 필요.

Co-Authored-By: Claude Sonnet 5 <noreply@anthropic.com>

File: ros2_ws/src/robot_arm_description/urdf/robot_arm.urdf (robot description, URDF)
Before this commit: robot robot_arm, 51 links, 50 joints
Links:
- removed link link_039
- added link link_051, mass 0.009342052845410124; collision mesh filename=package://robot_arm_description/meshes/link_051.stl scale=0.001 0.001 0.001; visual mesh filename=package://robot_arm_description/meshes/link_051.stl scale=0.001 0.001 0.001
- added link wrist_camera_link, mass 0.00012265625; collision mesh filename=package://robot_arm_description/meshes/wrist_camera_link.stl scale=0.001 0.001 0.001; visual mesh filename=package://robot_arm_description/meshes/wrist_camera_link.stl scale=0.001 0.001 0.001
- link base_link: mass 0.1213729503132452 -> 0.0940875583823606
- link link_001: mass 0.15394987554690048 -> 0.16917905697193936
- link link_002: mass 0.19814051788719486 -> 0.35060174014062084
- link link_003: mass 0.13969457823289902 -> 0.0024661502330680955
- link link_004: mass 0.27634623034311884 -> 0.09589711575082847
- link link_005: mass 0.28157202083896593 -> 0.05173873267885149
- link link_006: mass 0.08862458116688048 -> 0.05701847242477795
- link link_007: mass 0.08268035520095174 -> 0.5211129101861696
- link link_008: mass 0.07251339836837921 -> 0.025066272718870717
- link link_009: mass 0.07251339836837922 -> 0.16917905697193908
- link link_010: mass 0.19211177685064962 -> 0.00977563065213057
- link link_011: mass 0.19721325419288177 -> 0.07797742395878847
- link link_012: mass 0.21053904468872886 -> 0.07338537699525735
- link link_013: mass 0.10912049174690072 -> 0.03435402640600835
- link link_014: mass 0.016167745903671614 -> 0.024775801570545392
- link link_015: mass 0.006305281770624219 -> 0.026632124946508604
- link link_016: mass 1.2987414019147439 -> 0.07115250994468504
- link link_017: mass 1.2954622871398063 -> 0.0730419459973636
- link link_018: mass 0.01616774590367161 -> 0.1691790569719392
- link link_019: mass 0.10912049174690079 -> 0.032750599840462274
- link link_020: mass 0.020910021649792748 -> 0.016167745903671604
- link link_021: mass 0.02091002164979277 -> 1.0396025285523893
- link link_022: mass 0.024775801570545392 -> 0.021124136897098196
- link link_023: mass 0.10879656543491555 -> 0.1023504556826366
- link link_024: mass 0.03369324095260379 -> 0.05007124655260372
- link link_025: mass 0.026632124946508604 -> 0.03369324095260379
- link link_026: mass 0.03435402640600835 -> 0.026856814210510817
- link link_027: mass 0.013742837703337476 -> 0.10428593364406145
- link link_028: mass 0.12370727931856874 -> 0.03282391895069647
- link link_029: mass 0.1091204917469009 -> 0.02685681421051082
- link link_030: mass 0.0015707963267949652 -> 0.009497155157802643
- link link_031: mass 0.45227624478140094 -> 0.030622353778130273
- link link_032: mass 0.05007124655260372 -> 0.16867684563552796
- link link_033: mass 0.024380202336228632 -> 0.034085353103894385
- link link_034: mass 0.02073065249254581 -> 0.02130672512145345
- link link_035: mass 0.01887089370282533 -> 0.020920470983628755
- link link_036: mass 0.034085353103894385 -> 0.02073065249254581
- link link_037: mass 0.031236901804661328 -> 0.08821021033890361
- link link_038: mass 0.02374288789450661 -> 0.031236901804661328
- link link_040: mass 0.05689558566859283 -> 0.024380202336228632
- link link_041: mass 0.07583994930008672 -> 0.4873052897538753
- link link_042: mass 0.5057750603466008 -> 0.07583994930008672
- link link_043: mass 0.08821021033890362 -> 0.5057750603466008
- link link_044: mass 0.08821021033890375 -> 0.08821021033890362
- link link_045: mass 0.0034506939547765065 -> 0.08821021033890375
- link link_046: mass 0.0034506939547765073 -> 0.14107452059972816
- link link_047: mass 0.009342051864502975 -> 0.14107452059972586
- link link_048: mass 0.009342052845410124 -> 0.0034506939547765065
- link link_049: mass 0.14107452059972816 -> 0.0034506939547765073
- link link_050: mass 0.14107452059972586 -> 0.009342051864502975
Joints:
- added joint fixed_joint_042: type fixed, parent link_045, child link_049, origin xyz=-0.007999 -0.0039 -0.01175 rpy=0 0 0
- joint arm_joint_1: child link_028 -> link_004; limit effort=10.6 velocity=3.14159265358979 -> (none); origin xyz=0.0 0.0 0.04649999999999999 rpy=0.0 -0.0 0.0 -> xyz=0.0 0.0 0.0465 rpy=0 0 0; parent link_031 -> link_002
- joint arm_joint_2: axis 0.0 -0.0 -1.0 -> 1.0 0.0 0.0; child link_015 -> link_010; limit lower=0 upper=3.14159265358979 effort=106 velocity=0.314159265358979 -> lower=0.0 upper=3.141593 effort=100 velocity=100; origin xyz=0.0 0.0 -0.04650000000000001 rpy=0.0 -0.0 0.0 -> xyz=0.0465 0.0 0.0 rpy=0 0 0; parent link_013 -> link_009
- joint arm_joint_3: axis 0.0 0.0 -1.0 -> -1.0 0.0 -0.0; child link_021 -> link_022; limit lower=0 upper=3.14159265358979 effort=106 velocity=0.314159265358979 -> lower=0.0 upper=3.141593 effort=100 velocity=100; origin xyz=0.0 0.0 -0.07550000000000001 rpy=0.0 -0.0 0.0 -> xyz=-0.0755 0.0 0.0 rpy=0 0 0; parent link_017 -> link_021
- joint arm_joint_4: axis 0.0 2.6716461825402365e-33 -1.0 -> -1.0 0.0 0.0; child link_038 -> link_030; limit lower=-0.610865238198015 upper=0.872664625997165 effort=10.6 velocity=3.14159265358979 -> lower=-0.610865 upper=0.698132 effort=100 velocity=100; origin xyz=-0.0045 0.06891702 -0.0001 rpy=3.141592653589793 -0.0 3.141592653589793 -> xyz=0.0001 -0.068917 0.0045 rpy=0 0 0; parent link_006 -> link_028
- joint arm_joint_5: axis 0.0 -1.3358230912699144e-33 1.0 -> 0.0 -1.0 0.0; child link_033 -> link_040; limit effort=1.5 velocity=6.38790506229925 -> (none); origin xyz=-0.030900000000000004 0.005250000000000009 -0.0016439999999999977 rpy=-1.3358230912699144e-33 -4.09841728479371e-34 0.0 -> xyz=0.0309 0.001644 -0.00525 rpy=0 0 0; parent link_040 -> link_037
- joint fixed_joint_001: child link_029 -> link_001; origin xyz=0.0 0.01 0.004 rpy=0.0 -0.0 0.0 -> xyz=0.0 0.0 0.004 rpy=0 0 0
- joint fixed_joint_002: child link_031 -> link_002; origin xyz=0.0 0.01 0.004 rpy=0.0 -0.0 0.0 -> xyz=0.0 0.0 0.004 rpy=0 0 0
- joint fixed_joint_003: child link_030 -> link_003; origin xyz=0.0 0.0 0.04649999999999999 rpy=0.0 -0.0 0.0 -> xyz=0.0 0.0 0.0465 rpy=0 0 0; parent link_031 -> link_002
- joint fixed_joint_004: child link_003 -> link_005; origin xyz=0.0 0.0 0.0040000000000000036 rpy=0.0 -0.0 7.1287974851291655e-62 -> xyz=0.0 -0.01 0.0085 rpy=0 0 0; parent link_028 -> link_004
- joint fixed_joint_005: child link_001 -> link_006; origin xyz=0.0 0.0 0.0040000000000000036 rpy=3.141592653589793 -0.0 7.1287974851291655e-62 -> xyz=0.0 -0.01 0.0085 rpy=0 0 0; parent link_028 -> link_004
- joint fixed_joint_006: child link_016 -> link_007; origin xyz=0.06215 -0.00045606 0.05999999999999999 rpy=-3.141592653589793 -1.5707963267948966 0 -> xyz=-0.06215 0.004643 0.06 rpy=0 0 0; parent link_003 -> link_005
- joint fixed_joint_007: child link_014 -> link_008; origin xyz=0.0 -0.006000000000000001 -0.0675 rpy=0.0 -0.0 0.0 -> xyz=0.0675 -0.005731 0.0 rpy=0 0 0; parent link_016 -> link_007
- joint fixed_joint_008: child link_013 -> link_009; origin xyz=0.0 0.0 -0.010299999999999998 rpy=0.0 -0.0 0.0 -> xyz=0.0103 0.005544 -0.0045 rpy=0 0 0; parent link_014 -> link_008
- joint fixed_joint_009: child link_012 -> link_011; origin xyz=0.0 0.0 -0.014800000000000004 rpy=0.0 -0.0 0.0 -> xyz=0.0148 0.0 0.0 rpy=0 0 0; parent link_015 -> link_010
- joint fixed_joint_010: child link_002 -> link_012; origin xyz=-0.0009999999999999966 0.15 -0.001999999999999993 rpy=1.5707963267948966 -1.5707963267948966 0 -> xyz=0.002 0.15 -0.001 rpy=0 0 0; parent link_012 -> link_011
- joint fixed_joint_011: child link_022 -> link_013; origin xyz=0.001999999999999993 -0.061 -0.143 rpy=1.5707963267948966 -0.0 -1.5707963267948966 -> xyz=0.002 0.135652 0.049 rpy=0 0 0; parent link_002 -> link_011
- joint fixed_joint_012: child link_025 -> link_014; origin xyz=-0.002000000000000011 0.04699999999999999 -0.013818960000000012 rpy=-1.5707963267948966 -1.5707963267948966 0 -> xyz=-0.002 0.143 0.061 rpy=0 0 0; parent link_002 -> link_012
- joint fixed_joint_013: child link_026 -> link_015; origin xyz=0.04900000000000002 0.13565161 -0.001999999999999993 rpy=1.5707963267948966 -1.5707963267948966 0 -> xyz=0.002 0.013819 -0.047 rpy=0 0 0
- joint fixed_joint_014: child link_010 -> link_016; origin xyz=0.1586 0.0 -0.025 rpy=0.0 -0.0 0.0 -> xyz=-0.1586 0.025 0.0 rpy=0 0 0; parent link_026 -> link_013
- joint fixed_joint_015: child link_011 -> link_017; origin xyz=0.1586 0.0 0.0 rpy=3.141592653589793 -0.0 0.0 -> xyz=-0.1586 0.0 0.0 rpy=0 0 0; parent link_026 -> link_013
- joint fixed_joint_016: child link_020 -> link_018; origin xyz=0.001999999999999993 -0.04900000000000002 -0.13565161 rpy=-1.5707963267948966 -0.0 1.5707963267948966 -> xyz=-0.0303 0.0 0.0 rpy=0 0 0; parent link_011 -> link_014
- joint fixed_joint_017: origin xyz=0.0 0.0 -0.030300000000000004 rpy=0.0 -0.0 0.0 -> xyz=-0.002 -0.135652 -0.049 rpy=0 0 0; parent link_022 -> link_017
- joint fixed_joint_018: child link_018 -> link_020; origin xyz=0.0 0.0 -0.044000000000000004 rpy=0.0 -0.0 0.0 -> xyz=-0.044 0.0 0.0 rpy=0 0 0; parent link_019 -> link_018
- joint fixed_joint_019: child link_017 -> link_021; origin xyz=0.0 0.0 -0.04070000000000001 rpy=0.0 -0.0 0.0 -> xyz=-0.0407 0.0 0.0 rpy=0 0 0; parent link_018 -> link_020
- joint fixed_joint_020: child link_004 -> link_023; origin xyz=0.0 0.0 0.016500000000000004 rpy=3.141592653589793 -0.0 0.0 -> xyz=0.0165 0.0 0.0 rpy=0 0 0; parent link_021 -> link_022
- joint fixed_joint_021: child link_032 -> link_024; origin xyz=0.10800000000000001 -0.10673997 0.0 rpy=-1.5707963267948966 -0.0 -1.5707963267948966 -> xyz=0.0 -0.10674 0.108 rpy=0 0 0; parent link_004 -> link_023
- joint fixed_joint_022: child link_024 -> link_025; origin xyz=0.011999999999999993 -0.10673997 0.0 rpy=-1.5707963267948966 -0.0 1.5707963267948966 -> xyz=0.0 -0.10674 0.012 rpy=0 0 0; parent link_004 -> link_023
- joint fixed_joint_023: child link_008 -> link_026; origin xyz=0.06 -0.19462704 0.0 rpy=-1.5707963267948966 -0.0 0.0 -> xyz=0.0 -0.194627 0.06 rpy=0 0 0; parent link_004 -> link_023
- joint fixed_joint_024: child link_006 -> link_027; origin xyz=0.0 0.06865 0.0 rpy=-1.5707963267948966 5.473822126268817e-48 3.141592653589793 -> xyz=0.1943 0.0 0.0 rpy=0 0 0; parent link_008 -> link_024
- joint fixed_joint_025: child link_023 -> link_028; origin xyz=-0.004500000000000006 -0.0055439999999999864 0.003900000000000089 rpy=3.141592653589793 -0.0 0.0 -> xyz=0.06865 0.0 0.0 rpy=0 0 0; parent link_038 -> link_026
- joint fixed_joint_026: child link_036 -> link_029; origin xyz=0.006000000000000005 -0.0055439999999999864 -0.006699999999999907 rpy=0.0 -0.0 0.0 -> xyz=0.0 -0.087887 -0.048 rpy=0 0 0; parent link_038 -> link_027
- joint fixed_joint_027: child link_035 -> link_031; origin xyz=0.0035000000000000144 0.094 -0.005 rpy=0.0 -0.0 0.0 -> xyz=-0.06865 0.0 0.0 rpy=0 0 0; parent link_036 -> link_029
- joint fixed_joint_028: child link_034 -> link_032; origin xyz=-0.013000000000000008 0.094 -0.005 rpy=0.0 -0.0 0.0 -> xyz=0.0039 0.005544 -0.0045 rpy=0 0 0; parent link_036 -> link_030
- joint fixed_joint_029: child link_005 -> link_033; origin xyz=0.0 0.1943 0.0 rpy=3.141592653589793 -0.0 -3.141592653589793 -> xyz=-0.0067 0.005544 0.006 rpy=0 0 0; parent link_032 -> link_030
- joint fixed_joint_030: child link_009 -> link_034; origin xyz=-0.08788706999999998 0.0 0.04800000000000001 rpy=-3.141592653589793 -1.5707963267948966 0 -> xyz=0.0001 -0.068917 0.0045 rpy=0 0 0; parent link_005 -> link_031
- joint fixed_joint_031: child link_007 -> link_035; origin xyz=0.0 0.06865 0.0 rpy=-1.5707963267948966 5.473822126268817e-48 3.141592653589793 -> xyz=-0.005 -0.094 0.0035 rpy=0 0 0; parent link_009 -> link_033
- joint fixed_joint_032: child link_027 -> link_036; origin xyz=0.0 0.06337296 0.0 rpy=3.141592653589793 -0.0 0.0 -> xyz=-0.005 -0.094 -0.013 rpy=0 0 0; parent link_007 -> link_033
- joint fixed_joint_033: origin xyz=0.0 0.0 0.08190000000000001 rpy=0.0 -0.0 0.0 -> xyz=0.01505 -0.100544 -0.00025 rpy=0 0 0; parent link_035 -> link_033
- joint fixed_joint_034: child link_040 -> link_038; origin xyz=-0.0002499999999999845 0.100544 0.015050000000000003 rpy=-1.5707963267948966 1.5707963267948966 0 -> xyz=0.0819 0.0 0.0 rpy=0 0 0; parent link_036 -> link_035
- joint fixed_joint_035: child link_039 -> wrist_camera_link; origin xyz=0.0 0.0 0.005099999999999998 rpy=-3.141592653589793 1.1583765596690715e-32 -1.9721522630525295e-31 -> xyz=0.050523 -0.002178 0.061 rpy=0 0 0; parent link_033 -> link_035
- joint fixed_joint_036: origin xyz=0.0 0.0 -0.073 rpy=1.5707963267948966 0.0 -3.141592653589793 -> xyz=0.0 -0.0051 0.0 rpy=0 0 0; parent link_039 -> link_040
- joint fixed_joint_037: origin xyz=0.014 -0.005 0.018 rpy=0 0 0 -> xyz=0.0 -0.073 0.0 rpy=0 0 0
- joint fixed_joint_038: origin xyz=-0.002 -0.034 -0.007 rpy=0 0 0 -> xyz=0.014 -0.005 0.018 rpy=0 0 0
- joint fixed_joint_039: origin xyz=-0.026 -0.034 -0.007 rpy=0 0 0 -> xyz=-0.002 -0.034 -0.007 rpy=0 0 0; parent link_042 -> link_043
- joint fixed_joint_040: origin xyz=0.008001 -0.002 -0.010249 rpy=0 0 0 -> xyz=-0.026 -0.034 -0.007 rpy=0 0 0
- joint fixed_joint_041: child link_046 -> link_048; origin xyz=-0.007999 -0.0039 -0.01175 rpy=0 0 0 -> xyz=0.008001 -0.002 -0.010249 rpy=0 0 0
- joint gripper_left_pinion_joint: child link_047 -> link_050; parent link_045 -> link_048
- joint gripper_left_rack_joint: child link_049 -> link_046; parent link_042 -> link_043
- joint gripper_right_pinion_joint: child link_048 -> link_051; parent link_046 -> link_049
- joint gripper_right_rack_joint: child link_050 -> link_047; parent link_042 -> link_043
