Commit message: Checkpoint arm MoveIt pick-place and safe gripper change mode

File: ros2_ws/src/robot_arm_description/urdf/robot_arm.urdf (robot description, URDF)
Before this commit: robot robot_arm, 52 links, 51 joints
Joints:
- joint arm_joint_2: limit lower=0.0 upper=3.141593 effort=100 velocity=100 -> lower=-0.2 upper=3.141593 effort=100 velocity=100

Commit message: feat: add cleaner FSM and sensor abstraction

File: ros2_ws/src/robot_arm_description/urdf/robot_arm.urdf (robot description, URDF)
Before this commit: robot robot_arm, 58 links, 57 joints
Links:
- removed link link_042
- removed link link_043
- removed link link_044
- removed link link_045
- removed link link_046
- removed link link_047
- removed link link_048
- removed link link_049
- removed link link_050
- removed link link_052
- removed link link_053
- removed link link_054
- removed link link_055
- removed link link_056
- removed link link_057
- added link cleaner_base_link, mass 0.3359541709234757; collision mesh filename=package://robot_arm_description/meshes/cleaner_base_link.stl scale=0.001 0.001 0.001; visual mesh filename=package://robot_arm_description/meshes/cleaner_base_link.stl scale=0.001 0.001 0.001
Joints:
- removed joint fixed_joint_038
- removed joint fixed_joint_039
- removed joint fixed_joint_040
- removed joint gripper_drive_joint
- removed joint gripper_left_crank_joint
- removed joint gripper_left_finger_fixed
- removed joint gripper_left_inner_joint
- removed joint gripper_left_lower_jaw_joint
- removed joint gripper_left_upper_jaw_joint
- removed joint gripper_linkage_base_fixed
- removed joint gripper_right_crank_joint
- removed joint gripper_right_finger_fixed
- removed joint gripper_right_inner_joint
- removed joint gripper_right_lower_jaw_joint
- removed joint gripper_right_upper_jaw_joint
- added joint wrist_to_cleaner: type fixed, parent link_051, child cleaner_base_link, origin xyz=0 0 0 rpy=0 0 0

File: ros2_ws/src/robot_arm_description/urdf/robot_arm.urdf.xacro (robot description, xacro)
@@ -1,12 +1,10 @@
 <?xml version="1.0"?>
-<!-- 메인 xacro: robot_arm.urdf(2026-07-15 VerNOmiddle 통합 재export 기준, 팔+gripper_a 전체가
-     이미 하나의 tree)를 그대로 include. robot_arm.urdf는 <robot> 태그를 가진 완성 URDF지만,
+<!-- 메인 xacro: robot_arm.urdf(팔 5축 + link_051 아래 털털이 fixed base)를 그대로 include.
+     robot_arm.urdf는 <robot> 태그를 가진 완성 URDF지만,
      xacro:include는 루트 태그 이름과 무관하게 자식 엘리먼트를 그대로 이 파일의 <robot>에 이어붙임.
      이전엔 여기서 xacro:arg gripper로 그리퍼 모듈(urdf/grippers/*.xacro)을 골라 wrist_to_gripper
      fixed joint로 짜맞췄으나, 서로 다른 CAD export(팔/그리퍼 각각 다른 리비전)의 좌표계를 맞추는
      시도가 반복적으로 어긋나 폐기(2026-07-15, 사용자 결정) — robot_arm.urdf 헤더 주석 참고.
-     그리퍼 "모듈화"는 이제 로직 레벨(dynamixel_control의 gripper_type/gripper_presets.py)에서만
-     유지되고, URDF 레벨 스왑은 없음. 그리퍼를 실제로 교체하려면 robot_arm.urdf 자체를 새 통합
-     export로 다시 만들어야 함(urdf/grippers/ 디렉토리는 더 이상 사용 안 함). -->
+     털털이 ZIP에는 회전 joint가 없어서 회전축은 MoveIt 모델 밖의 별도 actuator로 둔다. -->
 <robot name="robot_arm" xmlns:xacro="http://www.ros.org/wiki/xacro">
   <xacro:include filename="$(find robot_arm_description)/urdf/robot_arm.urdf"/>

File: ros2_ws/src/robot_arm_moveit_config/config/robot_arm.ros2_control.xacro (robot description, xacro)
@@ -43,11 +43,4 @@
                 <state_interface name="velocity"/>
             </joint>
-            <joint name="gripper_drive_joint">
-                <command_interface name="position"/>
-                <state_interface name="position">
-                  <param name="initial_value">${initial_positions['gripper_drive_joint']}</param>
-                </state_interface>
-                <state_interface name="velocity"/>
-            </joint>
         </ros2_control>
     </xacro:macro>

Commit message: feat: integrate end-effector FSM and VLA interface

File: ros2_ws/src/robot_arm_description/urdf/robot_arm.urdf (robot description, URDF)
Before this commit: robot robot_arm, 44 links, 43 joints
Links:
- removed link cleaner_base_link
- added link ee_base_link, mass 0.3359541709234757; collision mesh filename=package://robot_arm_description/meshes/ee_description/base_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 scale=0.001 0.001 0.001; visual mesh filename=package://robot_arm_description/meshes/ee_description/base_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 scale=0.001 0.001 0.001
Joints:
- removed joint wrist_to_cleaner
- added joint wrist_to_ee: type fixed, parent link_051, child ee_base_link, origin xyz=0 0 0 rpy=0 0 0

File: ros2_ws/src/robot_arm_description/urdf/robot_arm.urdf.xacro (robot description, xacro)
@@ -1,4 +1,4 @@
 <?xml version="1.0"?>
-<!-- 메인 xacro: robot_arm.urdf(팔 5축 + link_051 아래 털털이 fixed base)를 그대로 include.
+<!-- 메인 xacro: robot_arm.urdf(팔 5축 + link_051 아래 ee_description fixed base)를 include.
      robot_arm.urdf는 <robot> 태그를 가진 완성 URDF지만,
      xacro:include는 루트 태그 이름과 무관하게 자식 엘리먼트를 그대로 이 파일의 <robot>에 이어붙임.
@@ -6,5 +6,6 @@
      fixed joint로 짜맞췄으나, 서로 다른 CAD export(팔/그리퍼 각각 다른 리비전)의 좌표계를 맞추는
      시도가 반복적으로 어긋나 폐기(2026-07-15, 사용자 결정) — robot_arm.urdf 헤더 주석 참고.
-     털털이 ZIP에는 회전 joint가 없어서 회전축은 MoveIt 모델 밖의 별도 actuator로 둔다. -->
+     ee_description.zip에는 joint/TCP가 전혀 없다. 따라서 MoveIt joint를 만들지 않으며,
+     별도 actuator는 하드웨어 사양이 주어질 때까지 fail-closed로 둔다. -->
 <robot name="robot_arm" xmlns:xacro="http://www.ros.org/wiki/xacro">
   <xacro:include filename="$(find robot_arm_description)/urdf/robot_arm.urdf"/>

File: ros2_ws/src/robot_arm_moveit_config/config/robot_arm.urdf.xacro (robot description, xacro)
@@ -2,5 +2,5 @@
 <robot xmlns:xacro="http://www.ros.org/wiki/xacro" name="robot_arm">
     <xacro:arg name="initial_positions_file" default="initial_positions.yaml" />
-    <!-- Import robot_arm urdf file (몸체 + gripper_a, robot_arm_description의 그리퍼 모듈화 xacro) -->
+    <!-- Import arm plus the fixed, single-link ee_description model. -->
     <xacro:include filename="$(find robot_arm_description)/urdf/robot_arm.urdf.xacro" />
     <!-- Import control_xacro -->
