Commit message: feat(arm): complete single-motor gripper pick-place integration

File: ros2_ws/src/robot_arm_description/urdf/robot_arm.urdf.xacro (robot description, xacro)
@@ -1,13 +1,16 @@
 <?xml version="1.0"?>
-<!-- 메인 xacro: robot_arm.urdf(2026-07-15 VerNOmiddle 통합 재export 기준, 팔+gripper_a 전체가
-     이미 하나의 tree)를 그대로 include. robot_arm.urdf는 <robot> 태그를 가진 완성 URDF지만,
-     xacro:include는 루트 태그 이름과 무관하게 자식 엘리먼트를 그대로 이 파일의 <robot>에 이어붙임.
-     이전엔 여기서 xacro:arg gripper로 그리퍼 모듈(urdf/grippers/*.xacro)을 골라 wrist_to_gripper
-     fixed joint로 짜맞췄으나, 서로 다른 CAD export(팔/그리퍼 각각 다른 리비전)의 좌표계를 맞추는
-     시도가 반복적으로 어긋나 폐기(2026-07-15, 사용자 결정) — robot_arm.urdf 헤더 주석 참고.
-     그리퍼 "모듈화"는 이제 로직 레벨(dynamixel_control의 gripper_type/gripper_presets.py)에서만
-     유지되고, URDF 레벨 스왑은 없음. 그리퍼를 실제로 교체하려면 robot_arm.urdf 자체를 새 통합
-     export로 다시 만들어야 함(urdf/grippers/ 디렉토리는 더 이상 사용 안 함). -->
+<!-- 엔드이펙터마다 검증된 통합 CAD export 전체를 선택한다. 서로 다른 export의 팔/그리퍼를
+     fixed joint로 추측 조립하지 않는다. dual은 현재 robot_arm.urdf, single은 git 3f048765에서
+     복원한 robot_arm.single_motor_gripper.urdf를 사용한다. -->
 <robot name="robot_arm" xmlns:xacro="http://www.ros.org/wiki/xacro">
-  <xacro:include filename="$(find robot_arm_description)/urdf/robot_arm.urdf"/>
+  <xacro:arg name="end_effector_preset" default="dual_motor_gripper"/>
+  <xacro:if value="${'$(arg end_effector_preset)' == 'dual_motor_gripper'}">
+    <xacro:include filename="$(find robot_arm_description)/urdf/robot_arm.urdf"/>
+  </xacro:if>
+  <xacro:if value="${'$(arg end_effector_preset)' == 'single_motor_gripper'}">
+    <xacro:include filename="$(find robot_arm_description)/urdf/robot_arm.single_motor_gripper.urdf"/>
+  </xacro:if>
+  <xacro:unless value="${'$(arg end_effector_preset)' in ['dual_motor_gripper', 'single_motor_gripper']}">
+    <xacro:include filename="$(find robot_arm_description)/urdf/robot_arm.urdf"/>
+  </xacro:unless>
 </robot>

File: ros2_ws/src/robot_arm_moveit_config/config/robot_arm.ros2_control.xacro (robot description, xacro)
@@ -1,5 +1,5 @@
 <?xml version="1.0"?>
 <robot xmlns:xacro="http://www.ros.org/wiki/xacro">
-    <xacro:macro name="robot_arm_ros2_control" params="name initial_positions_file">
+    <xacro:macro name="robot_arm_ros2_control" params="name initial_positions_file end_effector_preset">
         <xacro:property name="initial_positions" value="${load_yaml(initial_positions_file)['initial_positions']}"/>
         <ros2_control name="${name}" type="system">
@@ -43,11 +43,22 @@
                 <state_interface name="velocity"/>
             </joint>
-            <joint name="gripper_left_pinion_joint">
-                <command_interface name="position"/>
-                <state_interface name="position">
-                  <param name="initial_value">${initial_positions['gripper_left_pinion_joint']}</param>
-                </state_interface>
-                <state_interface name="velocity"/>
-            </joint>
+            <xacro:if value="${end_effector_preset == 'dual_motor_gripper'}">
+                <joint name="gripper_left_pinion_joint">
+                    <command_interface name="position"/>
+                    <state_interface name="position">
+                      <param name="initial_value">${initial_positions['gripper_left_pinion_joint']}</param>
+                    </state_interface>
+                    <state_interface name="velocity"/>
+                </joint>
+            </xacro:if>
+            <xacro:if value="${end_effector_preset == 'single_motor_gripper'}">
+                <joint name="gripper_drive_joint">
+                    <command_interface name="position"/>
+                    <state_interface name="position">
+                      <param name="initial_value">${initial_positions['gripper_drive_joint']}</param>
+                    </state_interface>
+                    <state_interface name="velocity"/>
+                </joint>
+            </xacro:if>
         </ros2_control>
     </xacro:macro>

File: ros2_ws/src/robot_arm_moveit_config/config/robot_arm.urdf.xacro (robot description, xacro)
@@ -2,8 +2,12 @@
 <robot xmlns:xacro="http://www.ros.org/wiki/xacro" name="robot_arm">
     <xacro:arg name="initial_positions_file" default="initial_positions.yaml" />
+    <xacro:arg name="end_effector_preset" default="dual_motor_gripper" />
     <!-- Import robot_arm urdf file (몸체 + gripper_a, robot_arm_description의 그리퍼 모듈화 xacro) -->
     <xacro:include filename="$(find robot_arm_description)/urdf/robot_arm.urdf.xacro" />
+    <xacro:property name="selected_end_effector_preset" value="$(arg end_effector_preset)"/>
     <!-- Import control_xacro -->
     <xacro:include filename="robot_arm.ros2_control.xacro" />
-    <xacro:robot_arm_ros2_control name="FakeSystem" initial_positions_file="$(arg initial_positions_file)"/>
+    <xacro:robot_arm_ros2_control name="FakeSystem"
+        initial_positions_file="$(arg initial_positions_file)"
+        end_effector_preset="$(arg end_effector_preset)"/>
 </robot>
